File: kicad/MODBUS.sch (KiCad schematic (older format))
At the start: 40 parts, among them J10 Conn_01x02, J11 Conn_01x02, J12 Conn_01x02, J13 Conn_01x02, J14 Screw_Terminal_01x02, J15 Screw_Terminal_01x02, J6 Conn_01x03, J7 Conn_01x03, J8 Conn_01x02, J9 Conn_01x02, U2 SN65HVD11, U3 SN65HVD11

Commit message: V0.2 Tapeout
Connections:
- net +3V3: now also D1.2 (A), D2.2 (A), D3.2 (A), D4.2 (A), R14.2, R16.2
- net GND: no longer D1.1 (K), D2.1 (K), D3.1 (K), D4.1 (K), R14.1, R16.1
- net RxD1: now also R14.1, R9.1; no longer R14.2, R9.2
- net RxD2: now also R10.1, R16.1; no longer R10.2, R16.2
- net TxD1: now also R7.1; no longer R7.2
- net TxD2: now also R8.1; no longer R8.2
- new net: D3.1 (K), R9.2
- new net: D1.1 (K), R7.2
- new net: D4.1 (K), R10.2
- new net: D2.1 (K), R8.2
Other:
- moved on the sheet: D1, D2, D3, D4, R10, R14, R16, R7, R8, R9
