File: kicad/rpi-atmega324-modbus-gateway-min.sch (KiCad schematic (older format))
At the start: 33 parts, among them J1 Raspberry_Pi_2+, J16 Conn_01x11, J17 Conn_01x11, J18 Conn_01x11, J19 Conn_01x11, J2 UART-Harwin3, J3 Conn_01x02, J4 Conn_02x03_Odd_Even, J5 Atmega-ISP-6, SW1 SW_Push, SW2 SW_SPST, U1 ATMEGA324P-20AU, Y1 12MHz

Commit message: V0.2 Tapeout
Parts:
- C2: value 100n -> 1n
Connections:
- wire segments 171 -> 172
- no-connect marks 30 -> 29
Changed lines of the file:
@@
 LIBS:contrib
 LIBS:valves
-LIBS:sx-atmega
-LIBS:sx-raspberry
-LIBS:sx-terminals
 LIBS:rpi-atmega324-modbus-gateway-min-cache
 EELAYER 25 0
@@
 Sheet 1 2
 Title "RPI Atmega324 Modbus Gateway"
-Date "2018-06-10"
-Rev "V0.1"
+Date "2018-08-30"
+Rev "V0.2"
 Comp "Manfred.Steiner@gmx.at"
 Comment1 ""
@@
 P 6450 1850
 F 0 "C2" H 6475 1950 50  0000 L CNN
-F 1 "100n" H 6475 1750 50  0000 L CNN
+F 1 "1n" H 6475 1750 50  0000 L CNN
 F 2 "Capacitors_SMD:C_1206_HandSoldering" H 6488 1700 50  0001 C CNN
 F 3 "" H 6450 1850 50  0001 C CNN
@@
 nSS
 NoConn ~ 10750 2200
-NoConn ~ 10750 2300
 $Comp
 L LED D7
@@
 	6000 5500 6200 5500
 Wire Wire Line
-	7100 4500 7100 6400
-Wire Wire Line
 	3400 5800 7100 5800
 Wire Wire Line
@@
 Wire Wire Line
 	3900 5100 3900 5000
-Wire Wire Line
-	7100 6400 5450 6400
-Connection ~ 7100 5800
-Wire Wire Line
-	6000 6300 6000 5600
 Wire Wire Line
 	6000 5600 6200 5600
@@
 	1    0    0    -1
 $EndComp
-Wire Wire Line
-	6000 6300 5450 6300
 $Comp
 L GND #PWR021
@@
 Text Notes 3650 7300 0    60   ~ 0
 Power Supply for standalone without Raspberry PI
+Wire Wire Line
+	10750 2300 10300 2300
+Text Label 10350 2300 0    60   ~ 0
+XTAL1
+Wire Wire Line
+	6000 5600 6000 6400
+Wire Wire Line
+	6000 6400 5450 6400
+Wire Wire Line
+	7100 4500 7100 6300
+Connection ~ 7100 5800
+Wire Wire Line
+	7100 6300 5450 6300
 $EndSCHEMATC
